File: kicad/simon.sch (KiCad schematic (older format))
At the start: 9 parts

Commit message: update
Parts:
- added C? (x2): 22 pF, symbol C
- added Y?: 16 MHz, symbol Crystal
- R? (x4): value R -> 1 KΩ
Connections:
- net Earth: now also IC?.22 (GND), IC?.8 (GND), C?.1, C?.1
- net at IC?.10 ((PCINT7/XTAL2/TOSC2)PB7): now also C?.2, Y?.2
- net +5V: now reaches IC?.20 (AVCC)
- net +5V: now also IC?.21 (AREF), IC?.7 (VCC)
- net at IC?.9 ((PCINT6/XTAL1/TOSC1)PB6): now also C?.2, Y?.1
Changed lines of the file:
@@
 P 6450 1400
 F 0 "R?" V 6530 1400 50  0000 C CNN
-F 1 "R" V 6450 1400 50  0000 C CNN
+F 1 "1 KΩ" V 6450 1400 50  0000 C CNN
 F 2 "" V 6380 1400 50  0000 C CNN
 F 3 "" H 6450 1400 50  0000 C CNN
@@
 P 6450 1700
 F 0 "R?" V 6530 1700 50  0000 C CNN
-F 1 "R" V 6450 1700 50  0000 C CNN
+F 1 "1 KΩ" V 6450 1700 50  0000 C CNN
 F 2 "" V 6380 1700 50  0000 C CNN
 F 3 "" H 6450 1700 50  0000 C CNN
@@
 P 6450 2000
 F 0 "R?" V 6530 2000 50  0000 C CNN
-F 1 "R" V 6450 2000 50  0000 C CNN
+F 1 "1 KΩ" V 6450 2000 50  0000 C CNN
 F 2 "" V 6380 2000 50  0000 C CNN
 F 3 "" H 6450 2000 50  0000 C CNN
@@
 P 6450 2300
 F 0 "R?" V 6530 2300 50  0000 C CNN
-F 1 "R" V 6450 2300 50  0000 C CNN
+F 1 "1 KΩ" V 6450 2300 50  0000 C CNN
 F 2 "" V 6380 2300 50  0000 C CNN
 F 3 "" H 6450 2300 50  0000 C CNN
@@
 	1    0    0    -1
 $EndComp
+$Comp
+L Crystal Y?
+U 1 1 5683CCD9
+P 4850 2100
+F 0 "Y?" H 4850 2250 50  0000 C CNN
+F 1 "16 MHz" H 4850 1950 50  0000 C CNN
+F 2 "" H 4850 2100 50  0000 C CNN
+F 3 "" H 4850 2100 50  0000 C CNN
+	1    4850 2100
+	0    1    1    0
+$EndComp
+$Comp
+L C C?
+U 1 1 5683CE46
+P 5350 2300
+F 0 "C?" H 5375 2400 50  0000 L CNN
+F 1 "22 pF" H 5375 2200 50  0000 L CNN
+F 2 "" H 5388 2150 50  0000 C CNN
+F 3 "" H 5350 2300 50  0000 C CNN
+	1    5350 2300
+	0    1    1    0
+$EndComp
+$Comp
+L C C?
+U 1 1 5683D0CC
+P 5350 1900
+F 0 "C?" H 5375 2000 50  0000 L CNN
+F 1 "22 pF" H 5375 1800 50  0000 L CNN
+F 2 "" H 5388 1750 50  0000 C CNN
+F 3 "" H 5350 1900 50  0000 C CNN
+	1    5350 1900
+	0    1    1    0
+$EndComp
+$Comp
+L Earth #PWR?
+U 1 1 5683D329
+P 5750 2100
+F 0 "#PWR?" H 5750 1850 50  0001 C CNN
+F 1 "Earth" H 5750 1950 50  0001 C CNN
+F 2 "" H 5750 2100 50  0000 C CNN
+F 3 "" H 5750 2100 50  0000 C CNN
+	1    5750 2100
+	0    -1   -1   0
+$EndComp
+$Comp
+L Earth #PWR?
+U 1 1 5683D79C
+P 1800 3950
+F 0 "#PWR?" H 1800 3700 50  0001 C CNN
+F 1 "Earth" H 1800 3800 50  0001 C CNN
+F 2 "" H 1800 3950 50  0000 C CNN
+F 3 "" H 1800 3950 50  0000 C CNN
+	1    1800 3950
+	1    0    0    -1
+$EndComp
+$Comp
+L +5V #PWR?
+U 1 1 5683D91E
+P 1800 1100
+F 0 "#PWR?" H 1800 950 50  0001 C CNN
+F 1 "+5V" H 1800 1240 50  0000 C CNN
+F 2 "" H 1800 1100 50  0000 C CNN
+F 3 "" H 1800 1100 50  0000 C CNN
+	1    1800 1100
+	1    0    0    -1
+$EndComp
 Wire Wire Line
 	6600 1400 6800 1400
@@
 Wire Wire Line
 	6000 2300 6300 2300
+Wire Wire Line
+	3950 1900 5200 1900
+Wire Wire Line
+	3950 2000 4550 2000
+Connection ~ 4850 1900
+Wire Wire Line
+	5600 1900 5500 1900
+Wire Wire Line
+	5600 2100 5750 2100
+Connection ~ 5600 2100
+Wire Wire Line
+	4850 1950 4850 1900
+Wire Wire Line
+	5600 1900 5600 2300
+Wire Wire Line
+	5600 2300 5500 2300
+Wire Wire Line
+	4550 2000 4550 2300
+Wire Wire Line
+	4550 2300 5200 2300
+Wire Wire Line
+	4850 2300 4850 2250
+Connection ~ 4850 2300
+Wire Wire Line
+	2050 3500 1800 3500
+Wire Wire Line
+	1800 3500 1800 3950
+Wire Wire Line
+	2050 3600 1800 3600
+Connection ~ 1800 3600
+Wire Wire Line
+	1800 1100 1800 1900
+Wire Wire Line
+	1800 1900 2050 1900
+Wire Wire Line
+	2050 1600 1800 1600
+Connection ~ 1800 1600
+Wire Wire Line
+	2050 1300 1800 1300
+Connection ~ 1800 1300
 $EndSCHEMATC

Commit message: update
Parts:
- added C?: 22pF, symbol C
- added R?: 1KΩ, symbol R
- added SP?: SPEAKER, symbol SPEAKER
- added SW?: Reset, symbol SW_PUSH
- IC?: value ATMEGA328-P -> ATMEGA328P-PU
- R? (x4): value 1 KΩ -> 470Ω
Connections:
- net +5V: now also R?.2
- net Earth: now also SP?.1, SW?.2
- net at IC?.1 ((PCINT14/~RESET~)PC6): now also C?.1, R?.1, SW?.1
- net Tx: now reaches IC?.2 ((PCINT16/RXD)PD0)
- net Rx: now reaches IC?.3 ((PCINT17/TXD)PD1)
- net at IC?.6 ((PCINT20/XCK/T0)PD4): now also SP?.2
- new net Reset: C?.2
Changed lines of the file:
@@
 P 2950 2400
 F 0 "IC?" H 2200 3650 50  0000 L BNN
-F 1 "ATMEGA328-P" H 3350 1000 50  0000 L BNN
+F 1 "ATMEGA328P-PU" H 3350 1000 50  0000 L BNN
 F 2 "DIL28" H 2950 2400 50  0000 C CIN
 F 3 "" H 2950 2400 50  0000 C CNN
@@
 P 6450 1400
 F 0 "R?" V 6530 1400 50  0000 C CNN
-F 1 "1 KΩ" V 6450 1400 50  0000 C CNN
+F 1 "470Ω" V 6450 1400 50  0000 C CNN
 F 2 "" V 6380 1400 50  0000 C CNN
 F 3 "" H 6450 1400 50  0000 C CNN
@@
 P 6450 1700
 F 0 "R?" V 6530 1700 50  0000 C CNN
-F 1 "1 KΩ" V 6450 1700 50  0000 C CNN
+F 1 "470Ω" V 6450 1700 50  0000 C CNN
 F 2 "" V 6380 1700 50  0000 C CNN
 F 3 "" H 6450 1700 50  0000 C CNN
@@
 P 6450 2000
 F 0 "R?" V 6530 2000 50  0000 C CNN
-F 1 "1 KΩ" V 6450 2000 50  0000 C CNN
+F 1 "470Ω" V 6450 2000 50  0000 C CNN
 F 2 "" V 6380 2000 50  0000 C CNN
 F 3 "" H 6450 2000 50  0000 C CNN
@@
 P 6450 2300
 F 0 "R?" V 6530 2300 50  0000 C CNN
-F 1 "1 KΩ" V 6450 2300 50  0000 C CNN
+F 1 "470Ω" V 6450 2300 50  0000 C CNN
 F 2 "" V 6380 2300 50  0000 C CNN
 F 3 "" H 6450 2300 50  0000 C CNN
@@
 L Earth #PWR?
 U 1 1 5682C917
-P 7600 2700
-F 0 "#PWR?" H 7600 2450 50  0001 C CNN
-F 1 "Earth" H 7600 2550 50  0001 C CNN
-F 2 "" H 7600 2700 50  0000 C CNN
-F 3 "" H 7600 2700 50  0000 C CNN
-	1    7600 2700
+P 7600 4350
+F 0 "#PWR?" H 7600 4100 50  0001 C CNN
+F 1 "Earth" H 7600 4200 50  0001 C CNN
+F 2 "" H 7600 4350 50  0000 C CNN
+F 3 "" H 7600 4350 50  0000 C CNN
+	1    7600 4350
 	1    0    0    -1
 $EndComp
@@
 $EndComp
 $Comp
-L Earth #PWR?
-U 1 1 5683D329
-P 5750 2100
-F 0 "#PWR?" H 5750 1850 50  0001 C CNN
-F 1 "Earth" H 5750 1950 50  0001 C CNN
-F 2 "" H 5750 2100 50  0000 C CNN
-F 3 "" H 5750 2100 50  0000 C CNN
-	1    5750 2100
-	0    -1   -1   0
-$EndComp
-$Comp
-L Earth #PWR?
-U 1 1 5683D79C
-P 1800 3950
-F 0 "#PWR?" H 1800 3700 50  0001 C CNN
-F 1 "Earth" H 1800 3800 50  0001 C CNN
-F 2 "" H 1800 3950 50  0000 C CNN
-F 3 "" H 1800 3950 50  0000 C CNN
-	1    1800 3950
-	1    0    0    -1
-$EndComp
-$Comp
 L +5V #PWR?
 U 1 1 5683D91E
-P 1800 1100
-F 0 "#PWR?" H 1800 950 50  0001 C CNN
-F 1 "+5V" H 1800 1240 50  0000 C CNN
-F 2 "" H 1800 1100 50  0000 C CNN
-F 3 "" H 1800 1100 50  0000 C CNN
-	1    1800 1100
-	1    0    0    -1
-$EndComp
+P 1800 800
+F 0 "#PWR?" H 1800 650 50  0001 C CNN
+F 1 "+5V" H 1800 940 50  0000 C CNN
+F 2 "" H 1800 800 50  0000 C CNN
+F 3 "" H 1800 800 50  0000 C CNN
+	1    1800 800
+	1    0    0    -1
+$EndComp
+$Comp
+L SPEAKER SP?
+U 1 1 5683EE28
+P 6400 3200
+F 0 "SP?" H 6300 3450 50  0000 C CNN
+F 1 "SPEAKER" H 6300 2950 50  0000 C CNN
+F 2 "" H 6400 3200 50  0000 C CNN
+F 3 "" H 6400 3200 50  0000 C CNN
+	1    6400 3200
+	1    0    0    -1
+$EndComp
+$Comp
+L R R?
+U 1 1 5683FEFD
+P 2950 900
+F 0 "R?" V 3030 900 50  0000 C CNN
+F 1 "1KΩ" V 2950 900 50  0000 C CNN
+F 2 "" V 2880 900 50  0000 C CNN
+F 3 "" H 2950 900 50  0000 C CNN
+	1    2950 900
+	0    1    1    0
+$EndComp
+$Comp
+L SW_PUSH SW?
+U 1 1 56840043
+P 4900 2750
+F 0 "SW?" H 5050 2860 50  0000 C CNN
+F 1 "Reset" H 4900 2670 50  0000 C CNN
+F 2 "" H 4900 2750 50  0000 C CNN
+F 3 "" H 4900 2750 50  0000 C CNN
+	1    4900 2750
+	1    0    0    -1
+$EndComp
+Text GLabel 4450 4500 3    60   Input ~ 0
+Reset
+Text GLabel 4300 4500 3    60   Input ~ 0
+Tx
+Text GLabel 4150 4500 3    60   Input ~ 0
+Rx
 Wire Wire Line
 	6600 1400 6800 1400
@@
 Wire Wire Line
 	6600 2300 6800 2300
-Wire Wire Line
-	7600 2700 7600 1400
 Wire Wire Line
 	7600 1400 7200 1400
@@
 Connection ~ 7600 1700
 Wire Wire Line
-	7200 2000 7600 2000
+	7600 2000 7200 2000
 Connection ~ 7600 2000
 Wire Wire Line
-	7200 2300 7600 2300
+	7600 2300 7200 2300
 Connection ~ 7600 2300
 Wire Wire Line
@@
 Connection ~ 1800 3600
 Wire Wire Line
-	1800 1100 1800 1900
+	1800 800  1800 1900
 Wire Wire Line
 	1800 1900 2050 1900
@@
 	2050 1300 1800 1300
 Connection ~ 1800 1300
+Wire Wire Line
+	5750 2100 5750 3100
+Wire Wire Line
+	7600 1400 7600 4350
+Wire Wire Line
+	5750 3100 6100 3100
+Wire Wire Line
+	6100 3300 3950 3300
+Wire Wire Line
+	1800 3950 7600 3950
+Connection ~ 7600 3950
+Wire Wire Line
+	1800 900  2800 900
+Connection ~ 1800 900
+Wire Wire Line
+	3100 900  4450 900
+Wire Wire Line
+	3950 2750 4600 2750
+Wire Wire Line
+	5200 2750 5750 2750
+Connection ~ 5750 2750
+Wire Wire Line
+	7600 2600 5750 2600
+Connection ~ 5750 2600
+Connection ~ 7600 2600
+Wire Wire Line
+	4300 2900 4300 4500
+Wire Wire Line
+	4150 3000 4150 4500
+$Comp
+L C C?
+U 1 1 56840AC3
+P 4450 4250
+F 0 "C?" H 4475 4350 50  0000 L CNN
+F 1 "22pF" H 4475 4150 50  0000 L CNN
+F 2 "" H 4488 4100 50  0000 C CNN
+F 3 "" H 4450 4250 50  0000 C CNN
+	1    4450 4250
+	1    0    0    -1
+$EndComp
+Wire Wire Line
+	3950 2900 4300 2900
+Wire Wire Line
+	3950 3000 4150 3000
+Wire Wire Line
+	4450 4500 4450 4400
+Wire Wire Line
+	4450 900  4450 4100
+Connection ~ 4450 2750
 $EndSCHEMATC

Commit message: update
Parts:
- added SW? (x4): SW_PUSH, symbol SW_PUSH
Connections:
- net Earth: now also SW?.2, SW?.2, SW?.2, SW?.2
- net at IC?.11 ((PCINT21/OC0B/T1)PD5): now also SW?.1
- net at IC?.12 ((PCINT22/OC0A/AIN0)PD6): now also SW?.1
- net at IC?.13 ((PCINT23/AIN1)PD7): now also SW?.1
- net at IC?.14 ((PCINT0/CLKO/ICP1)PB0): now also SW?.1
Changed lines of the file:
@@
 Text GLabel 4150 4500 3    60   Input ~ 0
 Rx
-Wire Wire Line
-	6600 1400 6800 1400
-Wire Wire Line
-	6600 1700 6800 1700
-Wire Wire Line
-	6600 2000 6800 2000
-Wire Wire Line
-	6600 2300 6800 2300
-Wire Wire Line
-	7600 1400 7200 1400
-Wire Wire Line
-	7200 1700 7600 1700
-Connection ~ 7600 1700
-Wire Wire Line
-	7600 2000 7200 2000
-Connection ~ 7600 2000
-Wire Wire Line
-	7600 2300 7200 2300
-Connection ~ 7600 2300
-Wire Wire Line
-	3950 1400 6300 1400
-Wire Wire Line
-	3950 1500 6200 1500
-Wire Wire Line
-	6200 1500 6200 1700
-Wire Wire Line
-	6200 1700 6300 1700
-Wire Wire Line
-	3950 1600 6100 1600
-Wire Wire Line
-	6100 1600 6100 2000
-Wire Wire Line
-	6100 2000 6300 2000
-Wire Wire Line
-	3950 1700 6000 1700
-Wire Wire Line
-	6000 1700 6000 2300
-Wire Wire Line
-	6000 2300 6300 2300
-Wire Wire Line
-	3950 1900 5200 1900
-Wire Wire Line
-	3950 2000 4550 2000
-Connection ~ 4850 1900
-Wire Wire Line
-	5600 1900 5500 1900
-Wire Wire Line
-	5600 2100 5750 2100
-Connection ~ 5600 2100
-Wire Wire Line
-	4850 1950 4850 1900
-Wire Wire Line
-	5600 1900 5600 2300
-Wire Wire Line
-	5600 2300 5500 2300
-Wire Wire Line
-	4550 2000 4550 2300
-Wire Wire Line
-	4550 2300 5200 2300
-Wire Wire Line
-	4850 2300 4850 2250
-Connection ~ 4850 2300
-Wire Wire Line
-	2050 3500 1800 3500
-Wire Wire Line
-	1800 3500 1800 3950
-Wire Wire Line
-	2050 3600 1800 3600
-Connection ~ 1800 3600
-Wire Wire Line
-	1800 800  1800 1900
-Wire Wire Line
-	1800 1900 2050 1900
-Wire Wire Line
-	2050 1600 1800 1600
-Connection ~ 1800 1600
-Wire Wire Line
-	2050 1300 1800 1300
-Connection ~ 1800 1300
-Wire Wire Line
-	5750 2100 5750 3100
-Wire Wire Line
-	7600 1400 7600 4350
-Wire Wire Line
-	5750 3100 6100 3100
-Wire Wire Line
-	6100 3300 3950 3300
-Wire Wire Line
-	1800 3950 7600 3950
-Connection ~ 7600 3950
-Wire Wire Line
-	1800 900  2800 900
-Connection ~ 1800 900
-Wire Wire Line
-	3100 900  4450 900
-Wire Wire Line
-	3950 2750 4600 2750
-Wire Wire Line
-	5200 2750 5750 2750
-Connection ~ 5750 2750
-Wire Wire Line
-	7600 2600 5750 2600
-Connection ~ 5750 2600
-Connection ~ 7600 2600
-Wire Wire Line
-	4300 2900 4300 4500
-Wire Wire Line
-	4150 3000 4150 4500
 $Comp
 L C C?
@@
 	1    0    0    -1
 $EndComp
+$Comp
+L SW_PUSH SW?
+U 1 1 56868A99
+P 5600 4300
+F 0 "SW?" H 5750 4410 50  0000 C CNN
+F 1 "SW_PUSH" H 5600 4220 50  0000 C CNN
+F 2 "" H 5600 4300 50  0000 C CNN
+F 3 "" H 5600 4300 50  0000 C CNN
+	1    5600 4300
+	1    0    0    -1
+$EndComp
+$Comp
+L SW_PUSH SW?
+U 1 1 56868C92
+P 5600 4700
+F 0 "SW?" H 5750 4810 50  0000 C CNN
+F 1 "SW_PUSH" H 5600 4620 50  0000 C CNN
+F 2 "" H 5600 4700 50  0000 C CNN
+F 3 "" H 5600 4700 50  0000 C CNN
+	1    5600 4700
+	1    0    0    -1
+$EndComp
+$Comp
+L SW_PUSH SW?
+U 1 1 56868D0A
+P 5600 5100
+F 0 "SW?" H 5750 5210 50  0000 C CNN
+F 1 "SW_PUSH" H 5600 5020 50  0000 C CNN
+F 2 "" H 5600 5100 50  0000 C CNN
+F 3 "" H 5600 5100 50  0000 C CNN
+	1    5600 5100
+	1    0    0    -1
+$EndComp
+$Comp
+L SW_PUSH SW?
+U 1 1 56868EC0
+P 5600 5500
+F 0 "SW?" H 5750 5610 50  0000 C CNN
+F 1 "SW_PUSH" H 5600 5420 50  0000 C CNN
+F 2 "" H 5600 5500 50  0000 C CNN
+F 3 "" H 5600 5500 50  0000 C CNN
+	1    5600 5500
+	1    0    0    -1
+$EndComp
+Wire Wire Line
+	6600 1400 6800 1400
+Wire Wire Line
+	6600 1700 6800 1700
+Wire Wire Line
+	6600 2000 6800 2000
+Wire Wire Line
+	6600 2300 6800 2300
+Wire Wire Line
+	7600 1400 7200 1400
+Wire Wire Line
+	7200 1700 7600 1700
+Connection ~ 7600 1700
+Wire Wire Line
+	7600 2000 7200 2000
+Connection ~ 7600 2000
+Wire Wire Line
+	7600 2300 7200 2300
+Connection ~ 7600 2300
+Wire Wire Line
+	3950 1400 6300 1400
+Wire Wire Line
+	3950 1500 6200 1500
+Wire Wire Line
+	6200 1500 6200 1700
+Wire Wire Line
+	6200 1700 6300 1700
+Wire Wire Line
+	3950 1600 6100 1600
+Wire Wire Line
+	6100 1600 6100 2000
+Wire Wire Line
+	6100 2000 6300 2000
+Wire Wire Line
+	3950 1700 6000 1700
+Wire Wire Line
+	6000 1700 6000 2300
+Wire Wire Line
+	6000 2300 6300 2300
+Wire Wire Line
+	3950 1900 5200 1900
+Wire Wire Line
+	3950 2000 4550 2000
+Connection ~ 4850 1900
+Wire Wire Line
+	5600 1900 5500 1900
+Wire Wire Line
+	5600 2100 5750 2100
+Connection ~ 5600 2100
+Wire Wire Line
+	4850 1950 4850 1900
+Wire Wire Line
+	5600 1900 5600 2300
+Wire Wire Line
+	5600 2300 5500 2300
+Wire Wire Line
+	4550 2000 4550 2300
+Wire Wire Line
+	4550 2300 5200 2300
+Wire Wire Line
+	4850 2300 4850 2250
+Connection ~ 4850 2300
+Wire Wire Line
+	2050 3500 1800 3500
+Wire Wire Line
+	1800 3500 1800 3950
+Wire Wire Line
+	2050 3600 1800 3600
+Connection ~ 1800 3600
+Wire Wire Line
+	1800 800  1800 1900
+Wire Wire Line
+	1800 1900 2050 1900
+Wire Wire Line
+	2050 1600 1800 1600
+Connection ~ 1800 1600
+Wire Wire Line
+	2050 1300 1800 1300
+Connection ~ 1800 1300
+Wire Wire Line
+	5750 2100 5750 3100
+Wire Wire Line
+	7600 1400 7600 4350
+Wire Wire Line
+	5750 3100 6100 3100
+Wire Wire Line
+	6100 3300 3950 3300
+Wire Wire Line
+	1800 3950 7600 3950
+Connection ~ 7600 3950
+Wire Wire Line
+	1800 900  2800 900
+Connection ~ 1800 900
+Wire Wire Line
+	3100 900  4450 900
+Wire Wire Line
+	3950 2750 4600 2750
+Wire Wire Line
+	5200 2750 5750 2750
+Connection ~ 5750 2750
+Wire Wire Line
+	7600 2600 5750 2600
+Connection ~ 5750 2600
+Connection ~ 7600 2600
+Wire Wire Line
+	4300 2900 4300 4500
+Wire Wire Line
+	4150 3000 4150 4500
 Wire Wire Line
 	3950 2900 4300 2900
@@
 	4450 900  4450 4100
 Connection ~ 4450 2750
+Wire Wire Line
+	5900 5500 6100 5500
+Wire Wire Line
+	6100 5500 6100 3950
+Connection ~ 6100 3950
+Wire Wire Line
+	5900 4300 6100 4300
+Connection ~ 6100 4300
+Wire Wire Line
+	5900 4700 6100 4700
+Connection ~ 6100 4700
+Wire Wire Line
+	5900 5100 6100 5100
+Connection ~ 6100 5100
+Wire Wire Line
+	3950 3400 5300 3400
+Wire Wire Line
+	5300 3400 5300 4300
+Wire Wire Line
+	3950 3500 5200 3500
+Wire Wire Line
+	5200 3500 5200 4700
+Wire Wire Line
+	5200 4700 5300 4700
+Wire Wire Line
+	3950 3600 5100 3600
+Wire Wire Line
+	5100 3600 5100 5100
+Wire Wire Line
+	5100 5100 5300 5100
+Wire Wire Line
+	3950 1300 4050 1300
+Wire Wire Line
+	4050 1300 4050 3700
+Wire Wire Line
+	4050 3700 5000 3700
+Wire Wire Line
+	5000 3700 5000 5500
+Wire Wire Line
+	5000 5500 5300 5500
 $EndSCHEMATC

Commit message: update
Parts:
- C2, C3: renamed from C?; value 22 pF -> 22pF
- Y1: renamed from Y?; value 16 MHz -> 16MHz
- gave numbers to parts that had none: 17
Changed lines of the file:
@@
 $EndDescr
 $Comp
-L ATMEGA328-P IC?
+L ATMEGA328-P IC1
 U 1 1 56819B05
 P 2950 2400
-F 0 "IC?" H 2200 3650 50  0000 L BNN
+F 0 "IC1" H 2200 3650 50  0000 L BNN
 F 1 "ATMEGA328P-PU" H 3350 1000 50  0000 L BNN
 F 2 "DIL28" H 2950 2400 50  0000 C CIN
@@
 $EndComp
 $Comp
-L LED D?
+L LED D1
 U 1 1 5682C58C
 P 7000 1400
-F 0 "D?" H 7000 1500 50  0000 C CNN
+F 0 "D1" H 7000 1500 50  0000 C CNN
 F 1 "LED" H 7000 1300 50  0000 C CNN
 F 2 "" H 7000 1400 50  0000 C CNN
@@
 $EndComp
 $Comp
-L LED D?
+L LED D2
 U 1 1 5682C66F
 P 7000 1700
-F 0 "D?" H 7000 1800 50  0000 C CNN
+F 0 "D2" H 7000 1800 50  0000 C CNN
 F 1 "LED" H 7000 1600 50  0000 C CNN
 F 2 "" H 7000 1700 50  0000 C CNN
@@
 $EndComp
 $Comp
-L LED D?
+L LED D3
 U 1 1 5682C6A8
 P 7000 2000
-F 0 "D?" H 7000 2100 50  0000 C CNN
+F 0 "D3" H 7000 2100 50  0000 C CNN
 F 1 "LED" H 7000 1900 50  0000 C CNN
 F 2 "" H 7000 2000 50  0000 C CNN
@@
 $EndComp
 $Comp
-L LED D?
+L LED D4
 U 1 1 5682C6DA
 P 7000 2300
-F 0 "D?" H 7000 2400 50  0000 C CNN
+F 0 "D4" H 7000 2400 50  0000 C CNN
 F 1 "LED" H 7000 2200 50  0000 C CNN
 F 2 "" H 7000 2300 50  0000 C CNN
@@
 $EndComp
 $Comp
-L R R?
+L R R2
 U 1 1 5682C700
 P 6450 1400
-F 0 "R?" V 6530 1400 50  0000 C CNN
+F 0 "R2" V 6530 1400 50  0000 C CNN
 F 1 "470Ω" V 6450 1400 50  0000 C CNN
 F 2 "" V 6380 1400 50  0000 C CNN
@@
 $EndComp
 $Comp
-L R R?
+L R R3
 U 1 1 5682C827
 P 6450 1700
-F 0 "R?" V 6530 1700 50  0000 C CNN
+F 0 "R3" V 6530 1700 50  0000 C CNN
 F 1 "470Ω" V 6450 1700 50  0000 C CNN
 F 2 "" V 6380 1700 50  0000 C CNN
@@
 $EndComp
 $Comp
-L R R?
+L R R4
 U 1 1 5682C85E
 P 6450 2000
-F 0 "R?" V 6530 2000 50  0000 C CNN
+F 0 "R4" V 6530 2000 50  0000 C CNN
 F 1 "470Ω" V 6450 2000 50  0000 C CNN
 F 2 "" V 6380 2000 50  0000 C CNN
@@
 $EndComp
 $Comp
-L R R?
+L R R5
 U 1 1 5682C890
 P 6450 2300
-F 0 "R?" V 6530 2300 50  0000 C CNN
+F 0 "R5" V 6530 2300 50  0000 C CNN
 F 1 "470Ω" V 6450 2300 50  0000 C CNN
 F 2 "" V 6380 2300 50  0000 C CNN
@@
 $EndComp
 $Comp
-L Earth #PWR?
+L Earth #PWR2
 U 1 1 5682C917
 P 7600 4350
-F 0 "#PWR?" H 7600 4100 50  0001 C CNN
+F 0 "#PWR2" H 7600 4100 50  0001 C CNN
 F 1 "Earth" H 7600 4200 50  0001 C CNN
 F 2 "" H 7600 4350 50  0000 C CNN
@@
 $EndComp
 $Comp
-L Crystal Y?
+L Crystal Y1
 U 1 1 5683CCD9
 P 4850 2100
-F 0 "Y?" H 4850 2250 50  0000 C CNN
-F 1 "16 MHz" H 4850 1950 50  0000 C CNN
+F 0 "Y1" H 4850 2250 50  0000 C CNN
+F 1 "16MHz" H 4850 1950 50  0000 C CNN
 F 2 "" H 4850 2100 50  0000 C CNN
 F 3 "" H 4850 2100 50  0000 C CNN
@@
 $EndComp
 $Comp
-L C C?
+L C C3
 U 1 1 5683CE46
 P 5350 2300
-F 0 "C?" H 5375 2400 50  0000 L CNN
-F 1 "22 pF" H 5375 2200 50  0000 L CNN
+F 0 "C3" H 5375 2400 50  0000 L CNN
+F 1 "22pF" H 5375 2200 50  0000 L CNN
 F 2 "" H 5388 2150 50  0000 C CNN
 F 3 "" H 5350 2300 50  0000 C CNN
@@
 $EndComp
 $Comp
-L C C?
+L C C2
 U 1 1 5683D0CC
 P 5350 1900
-F 0 "C?" H 5375 2000 50  0000 L CNN
-F 1 "22 pF" H 5375 1800 50  0000 L CNN
+F 0 "C2" H 5375 2000 50  0000 L CNN
+F 1 "22pF" H 5375 1800 50  0000 L CNN
 F 2 "" H 5388 1750 50  0000 C CNN
 F 3 "" H 5350 1900 50  0000 C CNN
@@
 $EndComp
 $Comp
-L +5V #PWR?
+L +5V #PWR1
 U 1 1 5683D91E
 P 1800 800
-F 0 "#PWR?" H 1800 650 50  0001 C CNN
+F 0 "#PWR1" H 1800 650 50  0001 C CNN
 F 1 "+5V" H 1800 940 50  0000 C CNN
 F 2 "" H 1800 800 50  0000 C CNN
@@
 $EndComp
 $Comp
-L SPEAKER SP?
+L SPEAKER SP1
 U 1 1 5683EE28
 P 6400 3200
-F 0 "SP?" H 6300 3450 50  0000 C CNN
+F 0 "SP1" H 6300 3450 50  0000 C CNN
 F 1 "SPEAKER" H 6300 2950 50  0000 C CNN
 F 2 "" H 6400 3200 50  0000 C CNN
@@
 $EndComp
 $Comp
-L R R?
+L R R1
 U 1 1 5683FEFD
 P 2950 900
-F 0 "R?" V 3030 900 50  0000 C CNN
+F 0 "R1" V 3030 900 50  0000 C CNN
 F 1 "1KΩ" V 2950 900 50  0000 C CNN
 F 2 "" V 2880 900 50  0000 C CNN
@@
 $EndComp
 $Comp
-L SW_PUSH SW?
+L SW_PUSH SW1
 U 1 1 56840043
 P 4900 2750
-F 0 "SW?" H 5050 2860 50  0000 C CNN
+F 0 "SW1" H 5050 2860 50  0000 C CNN
 F 1 "Reset" H 4900 2670 50  0000 C CNN
 F 2 "" H 4900 2750 50  0000 C CNN
@@
 Rx
 $Comp
-L C C?
+L C C1
 U 1 1 56840AC3
 P 4450 4250
-F 0 "C?" H 4475 4350 50  0000 L CNN
+F 0 "C1" H 4475 4350 50  0000 L CNN
 F 1 "22pF" H 4475 4150 50  0000 L CNN
 F 2 "" H 4488 4100 50  0000 C CNN
@@
 $EndComp
 $Comp
-L SW_PUSH SW?
+L SW_PUSH SW2
 U 1 1 56868A99
 P 5600 4300
-F 0 "SW?" H 5750 4410 50  0000 C CNN
+F 0 "SW2" H 5750 4410 50  0000 C CNN
 F 1 "SW_PUSH" H 5600 4220 50  0000 C CNN
 F 2 "" H 5600 4300 50  0000 C CNN
@@
 $EndComp
 $Comp
-L SW_PUSH SW?
+L SW_PUSH SW3
 U 1 1 56868C92
 P 5600 4700
-F 0 "SW?" H 5750 4810 50  0000 C CNN
+F 0 "SW3" H 5750 4810 50  0000 C CNN
 F 1 "SW_PUSH" H 5600 4620 50  0000 C CNN
 F 2 "" H 5600 4700 50  0000 C CNN
@@
 $EndComp
 $Comp
-L SW_PUSH SW?
+L SW_PUSH SW4
 U 1 1 56868D0A
 P 5600 5100
-F 0 "SW?" H 5750 5210 50  0000 C CNN
+F 0 "SW4" H 5750 5210 50  0000 C CNN
 F 1 "SW_PUSH" H 5600 5020 50  0000 C CNN
 F 2 "" H 5600 5100 50  0000 C CNN
@@
 $EndComp
 $Comp
-L SW_PUSH SW?
+L SW_PUSH SW5
 U 1 1 56868EC0
 P 5600 5500
-F 0 "SW?" H 5750 5610 50  0000 C CNN
+F 0 "SW5" H 5750 5610 50  0000 C CNN
 F 1 "SW_PUSH" H 5600 5420 50  0000 C CNN
 F 2 "" H 5600 5500 50  0000 C CNN
